File: hardware/SimpleFlightController.kicad_pcb (KiCad board)
At the start: 2 copper layers, 51.1 x 54.2 mm, 79 parts, among them J1 Screw_Terminal_01x02, J2 Conn_01x03, J3 Conn_01x03, SW1 TS-1088-AR02016, SW2 TS-1088-AR02016, U1 STM32F722RETx, U2 BQ25883RGER, U4 BMP580, U5 TPS63070RNMR, U6 LMR51430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

Commit message: Add files via upload
Parts:
- C3: footprint Capacitor_SMD:C_0603_1608Metric -> Capacitor_SMD:C_0805_2012Metric
Other:
- board text added: "Flight Controller by Naytik"
